File: caja_universal.sch (EAGLE design)
At the start: 45 parts, among them IC1 NE5534, IC2 AD620N, IC3 TL084P, IC4 TL084P, IC5 NE5534, IC6 TL072, T1 2N3904

Commit message: Corregidos valores circuito sense, potenciometro gain y cambio de libreria conectores. Agrego tRestrict alrededor de conectores para que las vias salgan siempre de bottom
Parts:
- removed +12V-FUSE, -12V-FUSE, HALL-PLACA, HR-PLACA, I-PLACA, LED, P-PLACA, T-PLACA: (no value), pinhead:PINHD-1X2
- removed POT-GAIN, POT-OFFSET, V-BAT, V-PLACA: (no value), pinhead:PINHD-1X3
- removed SWITCH-GRAL, SWITCH-P: (no value), pinhead:PINHD-1X4
- added J1: +12V-FUSE, con-molex:22-27-2021-02
- added J10: POT-OFFSET, con-molex:22-27-2031-03
- added J11: POT-GAIN, con-molex:22-27-2031-03
- added J12: I-PLACA, con-molex:22-27-2021-02
- added J13: SWITCH-P, con-molex:22-27-2041-04
- added J14: SWITCH-GRAL, con-molex:22-27-2041-04
- added J2: -12V-FUSE, con-molex:22-27-2021-02
- added J3: P-PLACA, con-molex:22-27-2021-02
- added J4: T-PLACA, con-molex:22-27-2021-02
- added J5: HR-PLACA, con-molex:22-27-2021-02
- added J6: HALL-PLACA, con-molex:22-27-2021-02
- added J7: LED, con-molex:22-27-2021-02
- added J8: V-PLACA, con-molex:22-27-2031-03
- added J9: V-BAT, con-molex:22-27-2031-03
- R16, R17: value 10k -> 1k
Connections:
- net +12V: now also IC6A.IN-, J1-2.S, J13-1.S, R14.1; no longer +12V-FUSE.2, IC6A.IN+, R14.2, SWITCH-P.1
- net +12VBAT: now also J14-2.S, J9-1.S; no longer SWITCH-GRAL.2, V-BAT.1
- net +12VFUSE: now also J1-1.S, J14-1.S; no longer +12V-FUSE.1, SWITCH-GRAL.1
- net +12VPLACA: now also IC6A.IN+, J8-1.S, R14.2; no longer IC6A.IN-, R14.1, V-PLACA.1
- net +I: now also J12-1.S; no longer I-PLACA.1
- net -1.25V: now also J10-1.S; no longer POT-OFFSET.3
- net -12V: now also J13-3.S, J2-2.S, J7-2.S, J8-3.S; no longer -12V-FUSE.2, LED.2, SWITCH-P.3, V-PLACA.3
- net -12VBAT: now also J14-4.S, J9-3.S; no longer SWITCH-GRAL.4, V-BAT.3
- net -12VFUSE: now also J14-3.S, J2-1.S; no longer -12V-FUSE.1, SWITCH-GRAL.3
- net -I: now also J12-2.S; no longer I-PLACA.2
- net 0V: now also J8-2.S, J9-2.S; no longer POT-GAIN.1, V-BAT.2, V-PLACA.2
- net 1.25V: now also J10-3.S; no longer POT-OFFSET.1
- net CHECK-LED: now also J7-1.S; no longer LED.1
- net HALL: now also J6-2.S; no longer HALL-PLACA.2
- net HR: now also J5-2.S; no longer HR-PLACA.2
- net N$16: now also J11-3.S; no longer POT-GAIN.3
- net OFFSET: now also J10-2.S; no longer POT-OFFSET.2
- net P+: now also J3-1.S; no longer P-PLACA.1
- net P-: now also J3-2.S; no longer P-PLACA.2
- net POUT: now also J11-2.S; no longer POT-GAIN.2
- net TENSION: now also J4-2.S; no longer T-PLACA.2
- net V+: now also J13-2.S; no longer SWITCH-P.2
- net V-: now also J13-4.S; no longer SWITCH-P.4
