File: mochila_full.sch (EAGLE design)
At the start: 13 parts, among them IC1 AD620R

Commit message: Agujeros de agarre del USB-C bien posicionados. No son agujeros, son PADS
Connections:
- net GND: now also USBC.PATA1, USBC.PATA2, USBC.PATA3, USBC.PATA4, USBC.PATA5, USBC.PATA6, USBC.PATA7, USBC.PATA8
- net OUTP-: now also FUJI.1
Changed lines of the file:
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@@
 <?xml version="1.0" encoding="utf-8"?>
 <!DOCTYPE eagle SYSTEM "eagle.dtd">
-<eagle version="7.7.0">
+<eagle version="9.2.2">
 <drawing>
 <settings>
 <setting alwaysvectorfont="no"/>
+<setting keepoldvectorfont="yes"/>
 <setting verticaltext="up"/>
 </settings>
@@
 </plain>
 <instances>
-<instance part="IC1" gate="G$1" x="60.96" y="58.42"/>
-<instance part="RG" gate="G$1" x="45.72" y="58.42" rot="R90"/>
-<instance part="C4" gate="G$1" x="22.86" y="48.26" rot="R90"/>
-<instance part="C3" gate="G$1" x="22.86" y="68.58" rot="R90"/>
-<instance part="R1" gate="G$1" x="38.1" y="38.1" rot="R270"/>
-<instance part="R2" gate="G$1" x="38.1" y="73.66" rot="R270"/>
-<instance part="VS" gate="G$1" x="-15.24" y="55.88"/>
-<instance part="FUJI" gate="G$1" x="104.14" y="78.74"/>
-<instance part="USBC" gate="G$1" x="129.54" y="25.4"/>
-<instance part="HALL" gate="A" x="93.98" y="27.94"/>
-<instance part="REG5V" gate="G$1" x="81.28" y="109.22"/>
-<instance part="C1" gate="G$1" x="63.5" y="104.14"/>
-<instance part="C2" gate="G$1" x="101.6" y="104.14"/>
+<instance part="IC1" gate="G$1" x="60.96" y="58.42" smashed="yes">
+<attribute name="NAME" x="69.85" y="64.77" size="1.778" layer="95"/>
+<attribute name="VALUE" x="69.85" y="50.8" size="1.778" layer="96"/>
+</instance>
+<instance part="RG" gate="G$1" x="45.72" y="58.42" smashed="yes" rot="R90">
+<attribute name="NAME" x="44.2214" y="54.61" size="1.778" layer="95" rot="R90"/>
+<attribute name="VALUE" x="49.022" y="54.61" size="1.778" layer="96" rot="R90"/>
+</instance>
+<instance part="C4" gate="G$1" x="22.86" y="48.26" smashed="yes" rot="R90">
+<attribute name="NAME" x="22.479" y="49.784" size="1.778" layer="95" rot="R90"/>
+<attribute name="VALUE" x="27.559" y="49.784" size="1.778" layer="96" rot="R90"/>
+</instance>
+<instance part="C3" gate="G$1" x="22.86" y="68.58" smashed="yes" rot="R90">
+<attribute name="NAME" x="22.479" y="70.104" size="1.778" layer="95" rot="R90"/>
+<attribute name="VALUE" x="27.559" y="70.104" size="1.778" layer="96" rot="R90"/>
+</instance>
+<instance part="R1" gate="G$1" x="38.1" y="38.1" smashed="yes" rot="R270">
+<attribute name="NAME" x="39.5986" y="41.91" size="1.778" layer="95" rot="R270"/>
+<attribute name="VALUE" x="34.798" y="41.91" size="1.778" layer="96" rot="R270"/>
+</instance>
+<instance part="R2" gate="G$1" x="38.1" y="73.66" smashed="yes" rot="R270">
+<attribute name="NAME" x="39.5986" y="77.47" size="1.778" layer="95" rot="R270"/>
+<attribute name="VALUE" x="34.798" y="77.47" size="1.778" layer="96" rot="R270"/>
+</instance>
+<instance part="VS" gate="G$1" x="-15.24" y="55.88" smashed="yes">
+<attribute name="NAME" x="-21.59" y="61.595" size="1.778" layer="95"/>
+<attribute name="VALUE" x="-21.59" y="50.8" size="1.778" layer="96"/>
+</instance>
+<instance part="FUJI" gate="G$1" x="104.14" y="78.74" smashed="yes">
+<attribute name="NAME" x="99.695" y="83.185" size="1.778" layer="95"/>
+<attribute name="VALUE" x="99.695" y="72.39" size="1.778" layer="96"/>
+</instance>
+<instance part="USBC" gate="G$1" x="129.54" y="25.4" smashed="yes">
+<attribute name="NAME" x="127" y="40.64" size="1.27" layer="95"/>
+<attribute name="VALUE" x="127" y="2.54" size="1.27" layer="96"/>
+</instance>
+<instance part="HALL" gate="A" x="93.98" y="27.94" smashed="yes">
+<attribute name="NAME" x="87.63" y="33.655" size="1.778" layer="95"/>
+<attribute name="VALUE" x="87.63" y="20.32" size="1.778" layer="96"/>
+</instance>
+<instance part="REG5V" gate="G$1" x="81.28" y="109.22" smashed="yes">
+<attribute name="NAME" x="76.2" y="114.935" size="1.778" layer="95"/>
+<attribute name="VALUE" x="76.2" y="112.395" size="1.778" layer="96"/>
+</instance>
+<instance part="C1" gate="G$1" x="63.5" y="104.14" smashed="yes">
+<attribute name="NAME" x="65.024" y="104.521" size="1.778" layer="95"/>
+<attribute name="VALUE" x="65.024" y="99.441" size="1.778" layer="96"/>
+</instance>
+<instance part="C2" gate="G$1" x="101.6" y="104.14" smashed="yes">
+<attribute name="NAME" x="103.124" y="104.521" size="1.778" layer="95"/>
+<attribute name="VALUE" x="103.124" y="99.441" size="1.778" layer="96"/>
+</instance>
 </instances>
 <busses>
@@
 <label x="81.28" y="91.44" size="1.778" layer="95"/>
 </segment>
+<segment>
+<pinref part="USBC" gate="G$1" pin="PATA1"/>
+<wire x1="116.84" y1="30.48" x2="109.22" y2="30.48" width="0.1524" layer="91"/>
+<label x="106.68" y="30.48" size="1.778" layer="95"/>
+</segment>
+<segment>
+<pinref part="USBC" gate="G$1" pin="PATA5"/>
+<wire x1="116.84" y1="25.4" x2="109.22" y2="25.4" width="0.1524" layer="91"/>
+<label x="106.68" y="25.4" size="1.778" layer="95"/>
+</segment>
+<segment>
+<pinref part="USBC" gate="G$1" pin="PATA7"/>
+<wire x1="116.84" y1="20.32" x2="114.3" y2="20.32" width="0.1524" layer="91"/>
+<wire x1="114.3" y1="20.32" x2="111.76" y2="20.32" width="0.1524" layer="91"/>
+<wire x1="111.76" y1="20.32" x2="109.22" y2="20.32" width="0.1524" layer="91"/>
+<label x="106.68" y="20.32" size="1.778" layer="95"/>
+</segment>
+<segment>
+<pinref part="USBC" gate="G$1" pin="PATA4"/>
+<wire x1="116.84" y1="15.24" x2="109.22" y2="15.24" width="0.1524" layer="91"/>
+<label x="106.68" y="15.24" size="1.778" layer="95"/>
+</segment>
+<segment>
+<pinref part="USBC" gate="G$1" pin="PATA2"/>
+<wire x1="193.04" y1="30.48" x2="203.2" y2="30.48" width="0.1524" layer="91"/>
+<label x="200.66" y="30.48" size="1.778" layer="95"/>
+</segment>
+<segment>
+<pinref part="USBC" gate="G$1" pin="PATA6"/>
+<wire x1="193.04" y1="25.4" x2="203.2" y2="25.4" width="0.1524" layer="91"/>
+<label x="200.66" y="25.4" size="1.778" layer="95"/>
+</segment>
+<segment>
+<pinref part="USBC" gate="G$1" pin="PATA8"/>
+<wire x1="193.04" y1="20.32" x2="203.2" y2="20.32" width="0.1524" layer="91"/>
+<label x="200.66" y="20.32" size="1.778" layer="95"/>
+</segment>
+<segment>
+<pinref part="USBC" gate="G$1" pin="PATA3"/>
+<wire x1="193.04" y1="15.24" x2="203.2" y2="15.24" width="0.1524" layer="91"/>
+<label x="200.66" y="15.24" size="1.778" layer="95"/>
+</segment>
 </net>
 <net name="N$5" class="0">
@@
 <wire x1="111.76" y1="81.28" x2="119.38" y2="81.28" width="0.1524" layer="91"/>
 <label x="119.38" y="81.28" size="1.778" layer="95"/>
-</segment>
-<segment>
+<pinref part="FUJI" gate="G$1" pin="1"/>
+<wire x1="96.52" y1="81.28" x2="96.52" y2="88.9" width="0.1524" layer="91"/>
+<wire x1="96.52" y1="88.9" x2="111.76" y2="88.9" width="0.1524" layer="91"/>
+<wire x1="111.76" y1="88.9" x2="111.76" y2="81.28" width="0.1524" layer="91"/>
+<junction x="111.76" y="81.28"/>
+</segment>
+<segment>
