File: caja_universal.brd (EAGLE design)
At the start: 45 parts, among them IC1 NE5534, IC2 AD620N, IC3 TL084P, IC4 TL084P, IC5 NE5534, IC6 TL072, J1 +12V-FUSE, J10 POT-OFFSET, J11 POT-GAIN, J12 I-PLACA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

Commit message: ...
Other:
- board outline added: 100 x 99 mm
